File: Hardware/specMech.brd (EAGLE design)
At the start: 142.2 x 121.9 mm, 64 parts, among them J1 PINHD-1X8-MOLEX-SHROUD, J2 Molex 0022232081, J3 PINHD-1X8-MOLEX-SHROUD, J4 PINHD-1X8-MOLEX-SHROUD, J5 XPORT, J6 Molex 0022232081, J7 Molex 0022232081, J8 Molex 0022232081, U1 MCP23008-E/SO, U10 ADS1115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

Commit message: Fixed level shifter orientation
Parts:
- moved C7 172.9 mm to (21.6, 100.3), flipped to the bottom, turned to 270 degrees
- moved C6 171.0 mm to (17.8, 99.7), flipped to the bottom, turned to 270 degrees
- moved C4 159.4 mm to (45.7, 118.7), flipped to the bottom, turned to 90 degrees
- moved R6 149.9 mm to (40.0, 98.4), flipped to the bottom, turned to 90 degrees
- moved R8 148.0 mm to (36.2, 98.4), flipped to the bottom, turned to 270 degrees
- moved R7 146.7 mm to (51.4, 98.4), flipped to the bottom, turned to 90 degrees
- moved C3 146.0 mm to (24.8, 97.8), flipped to the bottom, turned to 270 degrees
- moved C2 142.5 mm to (32.4, 98.4), flipped to the bottom, turned to 90 degrees
- moved R5 142.5 mm to (47.6, 98.4), flipped to the bottom, turned to 90 degrees
- moved C5 142.1 mm to (43.8, 101.0), flipped to the bottom, turned to 90 degrees
- moved U3 128.7 mm to (28.6, 98.4), flipped to the bottom
