File: Hardware/Eagle/specMech (2).brd (EAGLE design)
At the start: 142.2 x 121.9 mm, 82 parts, among them J1 PINHD-1X8-MOLEX-SHROUD, J2 Molex 0022232081, J3 PINHD-1X8-MOLEX-SHROUD, J4 PINHD-1X8-MOLEX-SHROUD, J5 XPORT, J6 Molex 0022232081, J7 Molex 0022232081, J8 Molex 0022232081, U1 MCP23008-E/SO, U10 ADS1115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

Commit message: Removed errant character at end of brd file
Parts:
- moved L3 6.48 mm to (92.7, 21.0)
- moved C12 5.08 mm to (107.3, 36.2)
- moved L1 5.08 mm to (110.5, 36.2)
- moved C1 5.08 mm to (108.0, 29.8)
- moved C14 5.08 mm to (104.1, 29.8)
- moved C15 5.08 mm to (100.3, 29.8)
- moved C16 5.08 mm to (96.5, 29.8)
- moved R16 5.08 mm to (111.8, 29.8)
- moved R22 5.08 mm to (99.7, 41.3)
- moved RN2 5.08 mm to (116.8, 29.8)
- moved U9 5.08 mm to (102.2, 34.9)
- moved R27 1.27 mm to (100.3, 16.5)
- moved C17 1.27 mm to (96.5, 6.99)
- moved C18 1.27 mm to (104.1, 6.99)
- moved C19 1.27 mm to (108.0, 6.99)
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