File: Hardware/Eagle/TerminalBlock.sch (EAGLE design)
At the start: 12 parts, among them J1 POWER TRANSFORMER, SW1 SPST-1437566-3

Commit message: Changed to 7-bit TWI addresses everywhere
Other:
- note added: "Pin R connector 3; Pin ? connector ? purple"
- note added: "To both motor controllers purple"
- note added: "To both motor controllers yellow"
- note removed: "Top motor controller"
Changed lines of the file:
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@@
 <setting verticaltext="up"/>
 </settings>
-<grid distance="0.1" unitdist="inch" unit="inch" style="lines" multiple="1" display="yes" altdistance="0.01" altunitdist="inch" altunit="inch"/>
+<grid distance="0.05" unitdist="inch" unit="inch" style="lines" multiple="1" display="yes" altdistance="0.01" altunitdist="inch" altunit="inch"/>
 <layers>
 <layer number="1" name="Top" color="4" fill="1" visible="no" active="no"/>
@@
 <text x="-17.78" y="-2.54" size="1.778" layer="150" rot="R180">Yellow</text>
 <text x="-17.78" y="10.16" size="1.778" layer="150" rot="R180">Red</text>
-<text x="38.1" y="-1.27" size="1.016" layer="150" rot="R180">Top motor controller</text>
+<text x="43.18" y="-1.27" size="1.016" layer="150" rot="R180">To both motor controllers yellow</text>
 <text x="-10.16" y="-8.89" size="1.016" layer="150" rot="R180">Pin X Connector 2</text>
 <text x="-20.32" y="-25.4" size="1.778" layer="150">Connectors are numbered
 from top to bottom 1-4</text>
+<text x="43.18" y="1.27" size="1.016" layer="150" rot="R180">To both motor controllers purple</text>
+<text x="50.8" y="3.81" size="1.016" layer="150" rot="R180">Pin R connector 3; Pin ? connector ? purple</text>
 </plain>
 <instances>
@@
 <junction x="10.16" y="2.54"/>
 <junction x="10.16" y="0"/>
-</segment>
-</net>
+<wire x1="15.24" y1="0" x2="22.86" y2="0" width="0.1524" layer="91"/>
+<junction x="15.24" y="0"/>
+<wire x1="15.24" y1="2.54" x2="22.86" y2="2.54" width="0.1524" layer="91"/>
+<junction x="15.24" y="2.54"/>
+</segment>
+</net>
