File: Hardware/Eagle/2021-03-30 specMech.sch (EAGLE design)
At the start: 91 parts, among them J1 PINHD-1X8-MOLEX-SHROUD, J10 MOLEX-22112022, J2 MOLEX-22112022, J3 PINHD-1X8-MOLEX-SHROUD, J4 PINHD-1X8-MOLEX-SHROUD, J5 Molex 22112042, J6 Molex 0022232081, J7 Lantronix XPORT, J8 Molex 0022232081, J9 MOLEX-22112022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

Commit message: Minor board edits
Parts:
- removed R7: 10K, AUmlib:R-US_R0805
Connections:
- removed net N$26: JP7.1, R6.1
- net +5V: now also JP7.1; no longer R6.2
- net GND: now also JP7.3; no longer R7.1
- net N$6: now also R6.1; no longer JP7.2
- net N$7: now also JP7.2, R6.2; no longer JP7.3, R7.2
Other:
- note added: "Spectrograph Number Select"
- note removed: "Spectrograph ID Select"
- moved on the sheet: JP7, R6
Changed lines of the file:
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@@
 <part name="C28" library="AUmlib" library_urn="urn:adsk.eagle:library:9166017" deviceset="C-US" device="C1210" package3d_urn="urn:adsk.eagle:package:4021267/2" value="10uF"/>
 <part name="GND50" library="AUmlib" library_urn="urn:adsk.eagle:library:9166017" deviceset="GND" device=""/>
-<part name="R7" library="AUmlib" library_urn="urn:adsk.eagle:library:9166017" deviceset="R-US_" device="R0805" package3d_urn="urn:adsk.eagle:package:4021199/4" value="10K"/>
 </parts>
 <sheets>
@@
 <description>Curiosity Nano</description>
 <plain>
-<text x="154.94" y="76.2" size="2.54" layer="250">Spectrograph
-ID Select</text>
+<text x="149.86" y="76.2" size="2.54" layer="250">Spectrograph
+Number Select</text>
 </plain>
 <instances>
@@
 <attribute name="DRAWING_NAME" x="190.5" y="19.05" size="2.54" layer="94"/>
 </instance>
-<instance part="JP7" gate="A" x="149.86" y="78.74" smashed="yes">
-<attribute name="NAME" x="143.51" y="84.455" size="1.778" layer="95"/>
-<attribute name="VALUE" x="143.51" y="71.12" size="1.778" layer="96"/>
+<instance part="JP7" gate="A" x="144.78" y="78.74" smashed="yes">
+<attribute name="NAME" x="138.43" y="84.455" size="1.778" layer="95"/>
+<attribute name="VALUE" x="138.43" y="71.12" size="1.778" layer="96"/>
 </instance>
-<instance part="R6" gate="G$1" x="139.7" y="88.9" smashed="yes" rot="R90">
-<attribute name="NAME" x="138.2014" y="87.63" size="1.778" layer="95" rot="R90"/>
-<attribute name="VALUE" x="143.002" y="87.63" size="1.778" layer="96" rot="R90"/>
+<instance part="R6" gate="G$1" x="127" y="78.74" smashed="yes">
+<attribute name="NAME" x="123.19" y="80.2386" size="1.778" layer="95"/>
+<attribute name="VALUE" x="123.19" y="75.438" size="1.778" layer="96"/>
 </instance>
-<instance part="P+28" gate="1" x="139.7" y="99.06" smashed="yes">
-<attribute name="VALUE" x="137.16" y="100.33" size="1.27" layer="96"/>
+<instance part="P+28" gate="1" x="134.62" y="86.36" smashed="yes">
+<attribute name="VALUE" x="132.08" y="87.63" size="1.27" layer="96"/>
 </instance>
-<instance part="GND43" gate="1" x="139.7" y="58.42" smashed="yes">
-<attribute name="VALUE" x="137.16" y="55.88" size="1.778" layer="96"/>
-</instance>
-<instance part="R7" gate="G$1" x="139.7" y="68.58" smashed="yes" rot="R90">
-<attribute name="NAME" x="138.2014" y="67.31" size="1.778" layer="95" rot="R90"/>
-<attribute name="VALUE" x="143.002" y="64.77" size="1.778" layer="96" rot="R90"/>
+<instance part="GND43" gate="1" x="134.62" y="71.12" smashed="yes">
+<attribute name="VALUE" x="132.08" y="68.58" size="1.778" layer="96"/>
 </instance>
 </instances>
@@
 </segment>
 <segment>
-<pinref part="R7" gate="G$1" pin="1"/>
 <pinref part="GND43" gate="1" pin="GND"/>
-<wire x1="139.7" y1="63.5" x2="139.7" y2="60.96" width="0.1524" layer="91"/>
+<wire x1="134.62" y1="73.66" x2="134.62" y2="76.2" width="0.1524" layer="91"/>
+<pinref part="JP7" gate="A" pin="3"/>
+<wire x1="134.62" y1="76.2" x2="142.24" y2="76.2" width="0.1524" layer="91"/>
 </segment>
 </net>
@@
 </segment>
 <segment>
+<pinref part="JP7" gate="A" pin="1"/>
+<wire x1="142.24" y1="81.28" x2="134.62" y2="81.28" width="0.1524" layer="91"/>
 <pinref part="P+28" gate="1" pin="+5V"/>
-<pinref part="R6" gate="G$1" pin="2"/>
-<wire x1="139.7" y1="96.52" x2="139.7" y2="93.98" width="0.1524" layer="91"/>
+<wire x1="134.62" y1="81.28" x2="134.62" y2="83.82" width="0.1524" layer="91"/>
 </segment>
 </net>
@@
 <wire x1="119.38" y1="132.08" x2="121.92" y2="132.08" width="0.1524" layer="91"/>
 <label x="121.92" y="132.08" size="1.016" layer="95" xref="yes"/>
+</segment>
+</net>
+<net name="N$6" class="0">
+<segment>
+<pinref part="CNANO1" gate="G$1" pin="PF2"/>
+<pinref part="R6" gate="G$1" pin="1"/>
+<wire x1="119.38" y1="78.74" x2="121.92" y2="78.74" width="0.1524" layer="91"/>
+</segment>
+</net>
+<net name="N$7" class="0">
+<segment>
+<pinref part="R6" gate="G$1" pin="2"/>
+<pinref part="JP7" gate="A" pin="2"/>
+<wire x1="132.08" y1="78.74" x2="142.24" y2="78.74" width="0.1524" layer="91"/>
 </segment>
 </net>
@@
 </segment>
 </net>
-<net name="N$26" class="0">
-<segment>
-<pinref part="JP7" gate="A" pin="1"/>
-<wire x1="147.32" y1="81.28" x2="139.7" y2="81.28" width="0.1524" layer="91"/>
-<pinref part="R6" gate="G$1" pin="1"/>
-<wire x1="139.7" y1="83.82" x2="139.7" y2="81.28" width="0.1524" layer="91"/>
-</segment>
-</net>
-<net name="N$6" class="0">
-<segment>
-<pinref part="JP7" gate="A" pin="2"/>
-<pinref part="CNANO1" gate="G$1" pin="PF2"/>
-<wire x1="147.32" y1="78.74" x2="119.38" y2="78.74" width="0.1524" layer="91"/>
-</segment>
-</net>
-<net name="N$7" class="0">
-<segment>
-<pinref part="JP7" gate="A" pin="3"/>
-<wire x1="139.7" y1="76.2" x2="147.32" y2="76.2" width="0.1524" layer="91"/>
-<pinref part="R7" gate="G$1" pin="2"/>
-<wire x1="139.7" y1="76.2" x2="139.7" y2="73.66" width="0.1524" layer="91"/>
-</segment>
-</net>
