File: Hardware/Eagle/2021-05-21 specMech.sch (EAGLE design)
At the start: 98 parts, among them J1 PINHD-1X8-MOLEX-SHROUD, J10 MOLEX-22112022, J11 POWER_JACKPJ-102AH, J2 MOLEX-22112022, J3 PINHD-1X8-MOLEX-SHROUD, J4 PINHD-1X8-MOLEX-SHROUD, J5 Molex 22112042, J6 Molex 0022232081, J7 Lantronix XPORT, J8 Molex 0022232081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

Commit message: Added get_MOTOR_LIMIT (not tested)
Other:
- note added: "Gold pin header Ion Pump Signals"
Changed lines of the file:
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@@
 <drawing>
 <settings>
-<setting alwaysvectorfont="yes"/>
+<setting alwaysvectorfont="no"/>
 <setting verticaltext="up"/>
 </settings>
-<grid distance="0.1" unitdist="inch" unit="inch" style="lines" multiple="1" display="no" altdistance="0.01" altunitdist="inch" altunit="inch"/>
+<grid distance="0.1" unitdist="inch" unit="inch" style="lines" multiple="1" display="yes" altdistance="0.01" altunitdist="inch" altunit="inch"/>
 <layers>
 <layer number="1" name="Top" color="4" fill="1" visible="no" active="no"/>
@@
 Pin 8 at 5.61, 0.83 in</text>
 <text x="160.02" y="139.7" size="1.778" layer="250">A3A is the AD590 connection</text>
+<text x="180.34" y="76.2" size="1.27" layer="250">Gold pin header
+Ion Pump Signals</text>
 </plain>
 <instances>
